File: KiCad_files/MusselGapeTracker_RevH/MusselGapeTracker_RevH.kicad_sch (KiCad schematic)
At the start: 83 parts, among them J1 AVR_SPI_PRG_6PTH, U1 ATMEGA328P, U2 DS3231M+TRL, U3 DS3231MZ

Commit message: Catching these up
Parts:
- MCP1700T-3302: symbol MusselGapeTracker_RevE-eagle-import:MCP1700T-3302E/TT -> MusselGapeTracker_RevE-eagle-import:MCP1700T-3302E/TT
Other:
- note added: "Designed by L.P. Miller, therefore use at your own risk"
